Commit message: urdf mesh paths

File: ur3e_robotiq/ur3e_robotiq_description/urdf/ur3e_robotiq.urdf (robot description, URDF)
Before this commit: robot ur3e_robotiq, 18 links, 17 joints
Links:
- link base_link_inertia: geometry collision mesh filename=file://$(find ur3e_robotiq_description)/urdf/meshes/collisi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; visual mesh filename=file://$(find ur3e_robotiq_description)/urdf/meshes/visual/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
- link forearm_link: geometry collision mesh filename=file://$(find ur3e_robotiq_description)/urdf/meshes/collisi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; visual mesh filename=file://$(find ur3e_robotiq_description)/urdf/meshes/visual/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
- link shoulder_link: geometry collision mesh filename=file://$(find ur3e_robotiq_description)/urdf/meshes/collisi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; visual mesh filename=file://$(find ur3e_robotiq_description)/urdf/meshes/visual/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
- link upper_arm_link: geometry collision mesh filename=file://$(find ur3e_robotiq_description)/urdf/meshes/collisi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; visual mesh filename=file://$(find ur3e_robotiq_description)/urdf/meshes/visual/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
- link wrist_1_link: geometry collision mesh filename=file://$(find ur3e_robotiq_description)/urdf/meshes/collisi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; visual mesh filename=file://$(find ur3e_robotiq_description)/urdf/meshes/visual/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
- link wrist_2_link: geometry collision mesh filename=file://$(find ur3e_robotiq_description)/urdf/meshes/collisi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; visual mesh filename=file://$(find ur3e_robotiq_description)/urdf/meshes/visual/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
- link wrist_3_link: geometry collision mesh filename=file://$(find ur3e_robotiq_description)/urdf/meshes/collisi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; visual mesh filename=file://$(find ur3e_robotiq_description)/urdf/meshes/visual/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
